Commit message: Simplify robot description

File: waldo_ros/waldo_description/urdf/kr16_2.xacro (robot description, xacro)
@@ -1,6 +1,288 @@
 <?xml version="1.0"?>
-<!--Generates a urdf from the macro in kr16_2_macro.xacro -->
 <robot name="kuka_kr16_2" xmlns:xacro="http://wiki.ros.org/xacro">
-  <xacro:include filename="$(find waldo_description)/urdf/kr16_2_macro.xacro" />
+  <!-- Define our robot as a macro so that we can provide parameters -->
+  <xacro:macro name="kuka_kr16_2" params="prefix">
+    <gazebo>
+      <plugin name="gazebo_ros_control" filename="libgazebo_ros_control.so">
+        <robotNamespace>/waldo</robotNamespace>
+        <robotSimType>gazebo_ros_control/DefaultRobotHWSim</robotSimType>
+      </plugin>
+    </gazebo>
+    <!-- Used for fixing robot to Gazebo 'base_link' -->
+    <link name="world"/>
+    <joint name="fixed" type="fixed">
+      <parent link="world"/>
+      <child link="base_link"/>
+    </joint>
+    <!-- LINKS -->
+    <!-- base link -->
+    <link name="${prefix}base_link">
+      <inertial>
+        <origin rpy="0 0 0" xyz="0 0 0"/>
+        <mass value="2"/>
+        <inertia ixx="0.01" ixy="0" ixz="0" iyy="0.01" iyz="0" izz="0.01"/>
+      </inertial>
+      <visual>
+        <origin xyz="0 0 0" rpy="0 0 0"/>
+        <geometry>
+          <mesh filename="package://waldo_description/meshes/kr16_2/visual/base_link.dae" />
+        </geometry>
+      </visual>
+      <collision>
+        <origin xyz="0 0 0" rpy="0 0 0"/>
+        <geometry>
+          <mesh filename="package://waldo_description/meshes/kr16_2/collision/base_link.stl" />
+        </geometry>
+      </collision>
+    </link>
+    <!-- link 1 (A1) -->
+    <link name="${prefix}link_1">
+      <inertial>
+        <origin xyz="0 0 0" rpy="0 0 0"/>
+        <mass value="2"/>
+        <inertia ixx="0.01" ixy="0" ixz="0" iyy="0.01" iyz="0" izz="0.01" />
+      </inertial>
+      <visual>
+        <origin xyz="0 0 0" rpy="0 0 0"/>
+        <geometry>
+          <mesh filename="package://waldo_description/meshes/kr16_2/visual/link_1.dae" />
+        </geometry>
+      </visual>
+      <collision>
+        <origin xyz="0 0 0" rpy="0 0 0"/>
+        <geometry>
+          <mesh filename="package://waldo_description/meshes/kr16_2/collision/link_1.stl" />
+        </geometry>
+      </collision>
+    </link>
+    <!-- link 2 -->
+    <link name="${prefix}link_2">
+      <inertial>
+        <origin xyz="0 0 0" rpy="0 0 0"/>
+        <mass value="2"/>
+        <inertia ixx="0.01" ixy="0" ixz="0" iyy="0.01" iyz="0" izz="0.01" />
+      </inertial>
+      <visual>
+        <origin xyz="0 0 0" rpy="0 0 0"/>
+        <geometry>
+          <mesh filename="package://waldo_description/meshes/kr16_2/visual/link_2.dae"/>
+        </geometry>
+      </visual>
+      <collision>
+        <origin xyz="0 0 0" rpy="0 0 0"/>
+        <geometry>
+          <mesh filename="package://waldo_description/meshes/kr16_2/collision/link_2.stl" />
+        </geometry>
+      </collision>
+    </link>
+    <!-- link 3 -->
+    <link name="${prefix}link_3">
+      <inertial>
+        <origin xyz="0 0 0" rpy="0 0 0"/>
+        <mass value="2"/>
+        <inertia ixx="0.01" ixy="0" ixz="0" iyy="0.01" iyz="0" izz="0.01" />
+      </inertial>
+      <visual>
+        <origin xyz="0 0 0" rpy="0 0 0"/>
+        <geometry>
+          <mesh filename="package://waldo_description/meshes/kr16_2/visual/link_3.dae" />
+        </geometry>
+      </visual>
+      <collision>
+        <origin xyz="0 0 0" rpy="0 0 0"/>
+        <geometry>
+          <mesh filename="package://waldo_description/meshes/kr16_2/collision/link_3.stl" />
+        </geometry>
+      </collision>
+    </link>
+    <!-- link 4 -->
+    <link name="${prefix}link_4">
+      <inertial>
+        <origin xyz="0 0 0" rpy="0 0 0"/>
+        <mass value="2"/>
+        <inertia ixx="0.01" ixy="0" ixz="0" iyy="0.01" iyz="0" izz="0.01" />
+      </inertial>
+      <visual>
+        <origin xyz="0 0 0" rpy="0 0 0"/>
+        <geometry>
+          <mesh filename="package://waldo_description/meshes/kr16_2/visual/link_4.dae" />
+        </geometry>
+      </visual>
+      <collision>
+        <origin xyz="0 0 0" rpy="0 0 0"/>
+        <geometry>
+          <mesh filename="package://waldo_description/meshes/kr16_2/collision/link_4.stl" />
+        </geometry>
+      </collision>
+    </link>
+    <!-- link 5 -->
+    <link name="${prefix}link_5">
+      <inertial>
+        <origin xyz="0 0 0" rpy="0 0 0"/>
+        <mass value="2"/>
+        <inertia ixx="0.01" ixy="0" ixz="0" iyy="0.01" iyz="0" izz="0.01" />
+      </inertial>
+      <visual>
+        <origin xyz="0 0 0" rpy="0 0 0"/>
+        <geometry>
+          <mesh filename="package://waldo_description/meshes/kr16_2/visual/link_5.dae" />
+        </geometry>
+      </visual>
+      <collision>
+        <origin xyz="0 0 0" rpy="0 0 0"/>
+        <geometry>
+          <mesh filename="package://waldo_description/meshes/kr16_2/collision/link_5.stl" />
+        </geometry>
+      </collision>
+    </link>
+    <!-- link 6 -->
+    <link name="${prefix}link_6">
+      <inertial>
+        <origin xyz="0 0 0" rpy="0 0 0"/>
+        <mass value="2"/>
+        <inertia ixx="0.01" ixy="0" ixz="0" iyy="0.01" iyz="0" izz="0.01" />
+      </inertial>
+      <visual>
+        <origin xyz="0 0 0" rpy="0 0 0"/>
+        <geometry>
+          <mesh filename="package://waldo_description/meshes/kr16_2/visual/link_6.dae" />
+        </geometry>
+      </visual>
+      <collision>
+        <origin xyz="0 0 0" rpy="0 0 0"/>
+        <geometry>
+          <mesh filename="package://waldo_description/meshes/kr16_2/collision/link_6.stl" />
+        </geometry>
+      </collision>
+    </link>
+    <!-- tool 0 -->
+    <!-- This frame corresponds to the $FLANGE coordinate system in KUKA KRC controllers. -->
+    <link name="${prefix}tool0"/>
+    <!-- END LINKS -->
+    <!-- JOINTS -->
+    <!-- joint 1 (A1) -->
+    <joint name="${prefix}joint_a1" type="revolute">
+      <origin xyz="0 0 0.675" rpy="0 0 0"/>
+      <parent link="${prefix}base_link"/>
+      <child link="${prefix}link_1"/>
+      <axis xyz="0 0 -1"/>
+      <limit effort="0" lower="${radians(-185)}" upper="${radians(185)}" velocity="${radians(156)}"/>
+    </joint>
+    <!-- joint 2 (A2) -->
+    <joint name="${prefix}joint_a2" type="revolute">
+      <origin xyz="0.26 0 0" rpy="0 0 0"/>
+      <parent link="${prefix}link_1"/>
+      <child link="${prefix}link_2"/>
+      <axis xyz="0 1 0"/>
+      <limit effort="0" lower="${radians(-155)}" upper="${radians(35)}" velocity="${radians(156)}"/>
+    </joint>
+    <!-- joint 3 (A3) -->
+    <joint name="${prefix}joint_a3" type="revolute">
+      <origin xyz="0.68 0 0" rpy="0 0 0"/>
+      <parent link="${prefix}link_2"/>
+      <child link="${prefix}link_3"/>
+      <axis xyz="0 1 0"/>
+      <limit effort="0" lower="${radians(-130)}" upper="${radians(154)}" velocity="${radians(156)}"/>
+    </joint>
+    <!-- joint 4 (A4) -->
+    <joint name="${prefix}joint_a4" type="revolute">
+      <origin xyz="0.67 0 -0.035" rpy="0 0 0"/>
+      <parent link="${prefix}link_3"/>
+      <child link="${prefix}link_4"/>
+      <axis xyz="-1 0 0"/>
+      <limit effort="0" lower="${radians(-350)}" upper="${radians(350)}" velocity="${radians(330)}"/>
+    </joint>
+    <!-- joint 5 (A5) -->
+    <joint name="${prefix}joint_a5" type="revolute">
+      <origin xyz="0 0 0" rpy="0 0 0"/>
+      <parent link="${prefix}link_4"/>
+      <child link="${prefix}link_5"/>
+      <axis xyz="0 1 0"/>
+      <limit effort="0" lower="${radians(-130)}" upper="${radians(130)}" velocity="${radians(330)}"/>
+    </joint>
+    <!-- joint 6 (A6) -->
+    <joint name="${prefix}joint_a6" type="revolute">
+      <origin xyz="0 0 0" rpy="0 0 0"/>
+      <parent link="${prefix}link_5"/>
+      <child link="${prefix}link_6"/>
+      <axis xyz="-1 0 0"/>
+      <limit effort="0" lower="${radians(-350)}" upper="${radians(350)}" velocity="${radians(615)}"/>
+    </joint>
+    <!-- tool frame - fixed frame -->
+    <joint name="${prefix}joint_a6-tool0" type="fixed">
+      <parent link="${prefix}link_6"/>
+      <child link="${prefix}tool0"/>
+      <origin xyz="0.158 0 0" rpy="0 ${radians(90)} 0"/>
+    </joint>
+    <!-- END JOINTS -->
+    <!-- ROS base_link to KUKA $ROBROOT coordinate system transform -->
+    <link name="${prefix}base" />
+    <joint name="${prefix}base_link-base" type="fixed">
+      <origin xyz="0 0 0" rpy="0 0 0"/>
+      <parent link="${prefix}base_link"/>
+      <child link="${prefix}base"/>
+    </joint>
+		<transmission name="trans_joint_a1">
+			<type>transmission_interface/SimpleTransmission</type>
+			<joint name="joint_a1">
+				<hardwareInterface>hardware_interface/JointStateInterface</hardwareInterface>
+			</joint>
+			<actuator name="joint_a1_motor">
+				<hardwareInterface>hardware_interface/JointStateInterface</hardwareInterface>
+				<mechanicalReduction>1</mechanicalReduction>
+			</actuator>
+		</transmission>
+		<transmission name="trans_joint_a2">
+			<type>transmission_interface/SimpleTransmission</type>
+			<joint name="joint_a2">
+				<hardwareInterface>hardware_interface/JointStateInterface</hardwareInterface>
+			</joint>
+			<actuator name="joint_a2_motor">
+				<hardwareInterface>hardware_interface/JointStateInterface</hardwareInterface>
+				<mechanicalReduction>1</mechanicalReduction>
+			</actuator>
+		</transmission>
+		<transmission name="trans_joint_a3">
+			<type>transmission_interface/SimpleTransmission</type>
+			<joint name="joint_a3">
+				<hardwareInterface>hardware_interface/JointStateInterface</hardwareInterface>
+			</joint>
+			<actuator name="joint_a3_motor">
+				<hardwareInterface>hardware_interface/JointStateInterface</hardwareInterface>
+				<mechanicalReduction>1</mechanicalReduction>
+			</actuator>
+		</transmission>
+		<transmission name="trans_joint_a4">
+			<type>transmission_interface/SimpleTransmission</type>
+			<joint name="joint_a4">
+				<hardwareInterface>hardware_interface/JointStateInterface</hardwareInterface>
+			</joint>
+			<actuator name="joint_a4_motor">
+				<hardwareInterface>hardware_interface/JointStateInterface</hardwareInterface>
+				<mechanicalReduction>1</mechanicalReduction>
+			</actuator>
+		</transmission>
+		<transmission name="trans_joint_a5">
+			<type>transmission_interface/SimpleTransmission</type>
+			<joint name="joint_a5">
+				<hardwareInterface>hardware_interface/JointStateInterface</hardwareInterface>
+			</joint>
+			<actuator name="joint_a5_motor">
+				<hardwareInterface>hardware_interface/JointStateInterface</hardwareInterface>
+				<mechanicalReduction>1</mechanicalReduction>
+			</actuator>
+		</transmission>
+		<transmission name="trans_joint_a6">
+			<type>transmission_interface/SimpleTransmission</type>
+			<joint name="joint_a6">
+				<hardwareInterface>hardware_interface/JointStateInterface</hardwareInterface>
+			</joint>
+			<actuator name="joint_a6_motor">
+				<hardwareInterface>hardware_interface/JointStateInterface</hardwareInterface>
+				<mechanicalReduction>1</mechanicalReduction>
+			</actuator>
+		</transmission>
+  </xacro:macro>
+  <!-- Call our robot macro defined above with the parameters defined -->
   <xacro:kuka_kr16_2 prefix=""/>
 </robot>

Commit message: Control KR 16 simulated in Gazebo

File: waldo_ros/waldo_description/urdf/kr16_2.xacro (robot description, xacro)
@@ -1,10 +1,71 @@
 <?xml version="1.0"?>
 <robot name="kuka_kr16_2" xmlns:xacro="http://wiki.ros.org/xacro">
+  <xacro:macro name="transmissions" params="hardwareInterface">
+		<transmission name="trans_joint_a1">
+			<type>transmission_interface/SimpleTransmission</type>
+			<joint name="joint_a1">
+				<hardwareInterface>${hardwareInterface}</hardwareInterface>
+			</joint>
+			<actuator name="joint_a1_motor">
+				<hardwareInterface>${hardwareInterface}</hardwareInterface>
+				<mechanicalReduction>1</mechanicalReduction>
+			</actuator>
+		</transmission>
+		<transmission name="trans_joint_a2">
+			<type>transmission_interface/SimpleTransmission</type>
+			<joint name="joint_a2">
+				<hardwareInterface>${hardwareInterface}</hardwareInterface>
+			</joint>
+			<actuator name="joint_a2_motor">
+				<hardwareInterface>${hardwareInterface}</hardwareInterface>
+				<mechanicalReduction>1</mechanicalReduction>
+			</actuator>
+		</transmission>
+		<transmission name="trans_joint_a3">
+			<type>transmission_interface/SimpleTransmission</type>
+			<joint name="joint_a3">
+				<hardwareInterface>${hardwareInterface}</hardwareInterface>
+			</joint>
+			<actuator name="joint_a3_motor">
+				<hardwareInterface>${hardwareInterface}</hardwareInterface>
+				<mechanicalReduction>1</mechanicalReduction>
+			</actuator>
+		</transmission>
+		<transmission name="trans_joint_a4">
+			<type>transmission_interface/SimpleTransmission</type>
+			<joint name="joint_a4">
+				<hardwareInterface>${hardwareInterface}</hardwareInterface>
+			</joint>
+			<actuator name="joint_a4_motor">
+				<hardwareInterface>${hardwareInterface}</hardwareInterface>
+				<mechanicalReduction>1</mechanicalReduction>
+			</actuator>
+		</transmission>
+		<transmission name="trans_joint_a5">
+			<type>transmission_interface/SimpleTransmission</type>
+			<joint name="joint_a5">
+				<hardwareInterface>${hardwareInterface}</hardwareInterface>
+			</joint>
+			<actuator name="joint_a5_motor">
+				<hardwareInterface>${hardwareInterface}</hardwareInterface>
+				<mechanicalReduction>1</mechanicalReduction>
+			</actuator>
+		</transmission>
+		<transmission name="trans_joint_a6">
+			<type>transmission_interface/SimpleTransmission</type>
+			<joint name="joint_a6">
+				<hardwareInterface>${hardwareInterface}</hardwareInterface>
+			</joint>
+			<actuator name="joint_a6_motor">
+				<hardwareInterface>${hardwareInterface}</hardwareInterface>
+				<mechanicalReduction>1</mechanicalReduction>
+			</actuator>
+		</transmission>
+  </xacro:macro>
   <!-- Define our robot as a macro so that we can provide parameters -->
   <xacro:macro name="kuka_kr16_2" params="prefix">
     <gazebo>
       <plugin name="gazebo_ros_control" filename="libgazebo_ros_control.so">
-        <robotNamespace>/waldo</robotNamespace>
-        <robotSimType>gazebo_ros_control/DefaultRobotHWSim</robotSimType>
+        <robotNamespace>/</robotNamespace>
       </plugin>
     </gazebo>
@@ -223,64 +284,6 @@
       <child link="${prefix}base"/>
     </joint>
-		<transmission name="trans_joint_a1">
-			<type>transmission_interface/SimpleTransmission</type>
-			<joint name="joint_a1">
-				<hardwareInterface>hardware_interface/JointStateInterface</hardwareInterface>
-			</joint>
-			<actuator name="joint_a1_motor">
-				<hardwareInterface>hardware_interface/JointStateInterface</hardwareInterface>
-				<mechanicalReduction>1</mechanicalReduction>
-			</actuator>
-		</transmission>
-		<transmission name="trans_joint_a2">
-			<type>transmission_interface/SimpleTransmission</type>
-			<joint name="joint_a2">
-				<hardwareInterface>hardware_interface/JointStateInterface</hardwareInterface>
-			</joint>
-			<actuator name="joint_a2_motor">
-				<hardwareInterface>hardware_interface/JointStateInterface</hardwareInterface>
-				<mechanicalReduction>1</mechanicalReduction>
-			</actuator>
-		</transmission>
-		<transmission name="trans_joint_a3">
-			<type>transmission_interface/SimpleTransmission</type>
-			<joint name="joint_a3">
-				<hardwareInterface>hardware_interface/JointStateInterface</hardwareInterface>
-			</joint>
-			<actuator name="joint_a3_motor">
-				<hardwareInterface>hardware_interface/JointStateInterface</hardwareInterface>
-				<mechanicalReduction>1</mechanicalReduction>
-			</actuator>
-		</transmission>
-		<transmission name="trans_joint_a4">
-			<type>transmission_interface/SimpleTransmission</type>
-			<joint name="joint_a4">
-				<hardwareInterface>hardware_interface/JointStateInterface</hardwareInterface>
-			</joint>
-			<actuator name="joint_a4_motor">
-				<hardwareInterface>hardware_interface/JointStateInterface</hardwareInterface>
-				<mechanicalReduction>1</mechanicalReduction>
-			</actuator>
-		</transmission>
-		<transmission name="trans_joint_a5">
-			<type>transmission_interface/SimpleTransmission</type>
-			<joint name="joint_a5">
-				<hardwareInterface>hardware_interface/JointStateInterface</hardwareInterface>
-			</joint>
-			<actuator name="joint_a5_motor">
-				<hardwareInterface>hardware_interface/JointStateInterface</hardwareInterface>
-				<mechanicalReduction>1</mechanicalReduction>
-			</actuator>
-		</transmission>
-		<transmission name="trans_joint_a6">
-			<type>transmission_interface/SimpleTransmission</type>
-			<joint name="joint_a6">
-				<hardwareInterface>hardware_interface/JointStateInterface</hardwareInterface>
-			</joint>
-			<actuator name="joint_a6_motor">
-				<hardwareInterface>hardware_interface/JointStateInterface</hardwareInterface>
-				<mechanicalReduction>1</mechanicalReduction>
-			</actuator>
-		</transmission>
+    <xacro:transmissions hardwareInterface="hardware_interface/PositionJointInterface"/>
+    <!--<xacro:transmissions hardwareInterface="hardware_interface/JointStateInterface">-->
   </xacro:macro>
   <!-- Call our robot macro defined above with the parameters defined -->
